Commit message: feat: 移植就绪 — URDF路径修复 + 机械臂集成 + 智能控制包 + 移植指南
- URDF file:// → package:// (26处, 跨平台兼容)
- robot_integrated.launch.py: 底盘+机械臂一体化启动
- robot_brain: 豆包语音对话、YOLO双目测距、视觉决策
- robot_desc_pub.py: TransientLocal 发布 /robot_description
- arm_full.launch.py: 机械臂一键启动
- serial_odom_receiver: 死区过滤+位置保持
- nav2_params: lifecycle超时15s
- PORTING_GUIDE.md: 完整移植文档

File: robot_ws/src/alloy_chassis_mecanum/urdf/alloy_chassis_mecanum.urdf (robot description, URDF)
Before this commit: robot 铝合金4驱底盘麦轮 -P1.STEP.SLDASM, 5 links, 4 joints
Links:
- link base_link: geometry collision mesh filename=package://alloy_chassis_mecanum/meshes/base_link.STL; visual mesh filename=package://alloy_chassis_mecanum/meshes/base_link.STL
- link wheel1_Link: geometry collision mesh filename=package://alloy_chassis_mecanum/meshes/wheel1_Link.STL; visual mesh filename=package://alloy_chassis_mecanum/meshes/wheel1_Link.STL
- link wheel2_Link: geometry collision mesh filename=package://alloy_chassis_mecanum/meshes/wheel2_Link.STL; visual mesh filename=package://alloy_chassis_mecanum/meshes/wheel2_Link.STL
- link wheel3_Link: geometry collision mesh filename=package://alloy_chassis_mecanum/meshes/wheel3_Link.STL; visual mesh filename=package://alloy_chassis_mecanum/meshes/wheel3_Link.STL
- link wheel4_Link: geometry collision mesh filename=package://alloy_chassis_mecanum/meshes/wheel4_Link.STL; visual mesh filename=package://alloy_chassis_mecanum/meshes/wheel4_Link.STL

File: robot_ws/src/arm_ros2/urdf/arm.urdf (robot description, URDF)
Before this commit: robot arm, 8 links, 7 joints
Links:
- link arm_Link1: geometry collision mesh filename=package://arm_ros2/meshes/arm_Link1.STL; visual mesh filename=package://arm_ros2/meshes/arm_Link1.STL
- link arm_Link2: geometry collision mesh filename=package://arm_ros2/meshes/arm_Link2.STL; visual mesh filename=package://arm_ros2/meshes/arm_Link2.STL
- link arm_Link3: geometry collision mesh filename=package://arm_ros2/meshes/arm_Link3.STL; visual mesh filename=package://arm_ros2/meshes/arm_Link3.STL
- link arm_Link4: geometry collision mesh filename=package://arm_ros2/meshes/arm_Link4.STL; visual mesh filename=package://arm_ros2/meshes/arm_Link4.STL
- link base_link: geometry collision mesh filename=package://arm_ros2/meshes/base_link.STL; visual mesh filename=package://arm_ros2/meshes/base_link.STL
- link end_Link1: geometry collision mesh filename=package://arm_ros2/meshes/end_Link1.STL; visual mesh filename=package://arm_ros2/meshes/end_Link1.STL
- link end_Link2: geometry collision mesh filename=package://arm_ros2/meshes/end_Link2.STL; visual mesh filename=package://arm_ros2/meshes/end_Link2.STL
- link gripper_Link: geometry collision mesh filename=package://arm_ros2/meshes/gripper_Link.STL; visual mesh filename=package://arm_ros2/meshes/gripper_Link.STL
