Commit message: feat: RDK X5 智能服务机器人 — 全功能集成版本
=== 新增功能 ===
- 模块化架构: navigator/grasper/detector 独立可测模块
- 一体化巡检抓取: integrated_patrol 导航→检测→抓取闭环
- 语音→动作全链路: voice_commander (Whisper + 豆包 Vision Pro)
- 果园智能分析: fruit_analyzer (HSV苹果质量分类) + cloud_uploader (火山引擎)
- 手眼标定: stereo_calibrate (双目棋盘格) + hand_eye_calibrate (ArUco+FK)
- IMU融合: serial_odom 0x03帧 + robot_localization EKF配置

=== 修复 ===
- robot_combined.urdf: 26处 file:// 绝对路径 → package://
- voice_chat.py: 移除硬编码API Key → 环境变量
- serial_odom_receiver: 默认端口 /dev/ttyUSB0 → /dev/ttyACM0
- yolo_stereo_detect: 删除开发机 sys.path hack
- run_moveit脚本: x86_64 Qt路径 → 自动检测架构
- 补全所有 CMakeLists.txt 和 package.xml 依赖声明

=== 文档 ===
- REPLICATION_GUIDE.md: 990行从零复刻教程
- PORTING_GUIDE.md: AI可执行的ARM64移植指南(10步+附录)
- 10篇调试日志 (logs/) 覆盖串口/Nav2/MoveIt/IMU/手眼标定/语音

Version: 2026-06-16 integrated release. Modules: navigator, grasper, detector, fruit_analyzer, cloud_uploader, voice_commander, integrated_patrol, orchard_patrol, hand_eye_calibrate, stereo_calibrate.

File: robot_ws/src/alloy_chassis_mecanum/urdf/robot_combined.urdf (robot description, URDF)
Before this commit: robot 铝合金4驱底盘麦轮 -P1.STEP.SLDASM, 13 links, 12 joints
Links:
- link arm_Link1: geometry collision mesh filename=package://arm_ros2/meshes/arm_Link1.STL; visual mesh filename=package://arm_ros2/meshes/arm_Link1.STL
- link arm_Link2: geometry collision mesh filename=package://arm_ros2/meshes/arm_Link2.STL; visual mesh filename=package://arm_ros2/meshes/arm_Link2.STL
- link arm_Link3: geometry collision mesh filename=package://arm_ros2/meshes/arm_Link3.STL; visual mesh filename=package://arm_ros2/meshes/arm_Link3.STL
- link arm_Link4: geometry collision mesh filename=package://arm_ros2/meshes/arm_Link4.STL; visual mesh filename=package://arm_ros2/meshes/arm_Link4.STL
- link arm_base_link: geometry collision mesh filename=package://arm_ros2/meshes/base_link.STL; visual mesh filename=package://arm_ros2/meshes/base_link.STL
- link base_link: geometry collision mesh filename=package://alloy_chassis_mecanum/meshes/base_link.STL; visual mesh filename=package://alloy_chassis_mecanum/meshes/base_link.STL
- link end_Link1: geometry collision mesh filename=package://arm_ros2/meshes/end_Link1.STL; visual mesh filename=package://arm_ros2/meshes/end_Link1.STL
- link end_Link2: geometry collision mesh filename=package://arm_ros2/meshes/end_Link2.STL; visual mesh filename=package://arm_ros2/meshes/end_Link2.STL
- link gripper_Link: geometry collision mesh filename=package://arm_ros2/meshes/gripper_Link.STL; visual mesh filename=package://arm_ros2/meshes/gripper_Link.STL
- link wheel1_Link: geometry collision mesh filename=package://alloy_chassis_mecanum/meshes/wheel1_Link.STL; visual mesh filename=package://alloy_chassis_mecanum/meshes/wheel1_Link.STL
- link wheel2_Link: geometry collision mesh filename=package://alloy_chassis_mecanum/meshes/wheel2_Link.STL; visual mesh filename=package://alloy_chassis_mecanum/meshes/wheel2_Link.STL
- link wheel3_Link: geometry collision mesh filename=package://alloy_chassis_mecanum/meshes/wheel3_Link.STL; visual mesh filename=package://alloy_chassis_mecanum/meshes/wheel3_Link.STL
- link wheel4_Link: geometry collision mesh filename=package://alloy_chassis_mecanum/meshes/wheel4_Link.STL; visual mesh filename=package://alloy_chassis_mecanum/meshes/wheel4_Link.STL
